File: dMarkle.kicad_sch (KiCad schematic)
At the start: 61 parts, among them SW1 SW_Choice, U1 74LS125, U10 INND-TS30RCB, U2 74HC4511, U3 Pico, U4 INND-TS30RCB, U5 74LS125, U6 74LS125, U7 74HC4511, U8 74HC4511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

Commit message: Add another LS125 for rotary encoder output.
Parts:
- added C15: 1u, Capacitor_THT:CP_Radial_D5.0mm_P2.00mm, symbol Device:C_Polarized_Small
- added C16: 0u1, Capacitor_THT:C_Rect_L4.0mm_W2.5mm_P2.50mm, symbol Device:C_Small
- added U11: 74LS125, Package_DIP:DIP-14_W7.62mm, symbol 74xx:74LS125
- SW1: Manufacturer (none) -> Bourns Inc.; Manufacturer Part Number (none) -> PEC12R-4220F-S0024; Supplier Part Number (none) -> PEC12R-4220F-S0024-ND
Connections:
- net +3.3V: now also U11.14 (VCC); no longer R3.1, R4.1, R5.1
- net +5V: now also R3.1, R4.1, R5.1, C15.1, C16.1
- net GND: now also C15.2, C16.2, U11.1, U11.10, U11.4, U11.7 (GND)
- net R_CLK: now also U11.3; no longer R1.1
- net R_DT: now also U11.6; no longer R2.1
- net R_~{SW}: now also U11.8; no longer C17.1, R6.2
- new net: C17.1, R6.2, U11.9
- new net: R1.1, U11.2
- new net: R2.1, U11.5
- no-connect marks 19 -> 22
Other:
- moved on the sheet: C17, C5, C8, R1, R2, R3, R4, R5, R6, SW1, U3
