File: dMarkle_Bottom/dMarkle_Bottom.kicad_pcb (KiCad board)
At the start: 2 copper layers, 86.4 x 75.1 mm, 29 parts, among them J1 HDR_Output, J2 HDR_Input, U1 Pico, U2 74HC125, U3 74HC125, U4 74HC125, U5 74HC125

Commit message: Initial split of dMarkle board
Parts:
- added Q1: Q_NJFET_DGS, Package_TO_SOT_THT:TO-220-3_Horizontal_TabUp, F.Cu at (107.6, 60.7)
- moved D2 44.5 mm to (167.4, 58.7)
- moved R6 44.2 mm to (169.7, 57.7)
- moved D1 39.6 mm to (167.4, 53.8)
- moved R1 39.5 mm to (169.7, 52.8)
- moved C2 16.0 mm to (131.1, 53.1), turned to 0 degrees
- moved C1 10.7 mm to (113.0, 48.5)
Connections:
- U1 pad 39: +5V -> /VBUS
- U1 pad 40: +5V -> /VBUS
Routing:
- net +5V: track 169.3 -> 0.01 mm, vias 2 -> 0
- net 3V3_EN: track 48.3 -> 62.2 mm
- net +3.3V: track 110.8 -> 116.4 mm
- net ~{RESET}: track 31.1 -> 29.1 mm
- net /IBA.D1: track 36.2 -> 35.2 mm
- net /IBA.D2: track 42.4 -> 41.5 mm
- net /IA.D0: track 52.1 -> 51.3 mm
- net /OBA.~{OE}: track 45.6 -> 44.8 mm
- net /OBB.~{OE}: track 53.5 -> 52.8 mm
- net /OBC.~{OE}: track 51.8 -> 51.0 mm
- net GND: vias 9 -> 0
- added copper zone on F.Cu, net /VBUS
- removed copper zone on F.Cu, net GND
Other:
- board text added: "3V3"
- board text added: "3V3_EN"
- board text added: "5V"
- board text added: "D0"
- board text added: "D1"
- board text added: "D2"
- board text added: "D3"
- board text added: "GND"
- board text added: "Input A"
- board text added: "~{RESET}"
